File: PCB/Volumeter.sch (KiCad schematic (older format))
At the start: 11 parts, among them SW1 SW_Push, U1 ATtiny85-20PU

Commit message: renamed project to volumeter
Parts:
- C1: footprint Capacitor_THT:CP_Radial_D4.0mm_P2.00mm -> Capacitor_THT:CP_Radial_D5.0mm_P2.50mm
Changed lines of the file:
@@
 F 0 "C1" H 6515 1196 50  0000 L CNN
 F 1 "100uF" H 6515 1105 50  0000 L CNN
-F 2 "Capacitor_THT:CP_Radial_D4.0mm_P2.00mm" H 6438 1000 50  0001 C CNN
+F 2 "Capacitor_THT:CP_Radial_D5.0mm_P2.50mm" H 6438 1000 50  0001 C CNN
 F 3 "~" H 6400 1150 50  0001 C CNN
 	1    6400 1150
